File: SensorTemperatura.sch (EAGLE design)
At the start: 14 parts, among them IC1 MAX481CPA, IC2 MEGA8-P

Commit message: add changes
Parts:
- added S2: (no value), switch-omron:10-XX
- added X1: (no value), con-ptr500:AK500/2
- added X2, X3: (no value), con-ptr500:AK500/3
Connections:
- new net N$10: IC2.PD3(INT1), X2-2.KL
- new net N$15: IC1G$1.B, X3-3.KL
- new net N$16: IC1G$1.A, X3-2.KL
- net GND: now also S2.S, S2.S1, X1-1.KL, X2-1.KL, X3-1.KL
- net N$13: now also S2.P, S2.P1
- net VCC: now also X1-2.KL, X2-3.KL
Changed lines of the file:
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@@
 <part name="P+5" library="supply1" deviceset="VCC" device=""/>
 <part name="GND4" library="supply1" deviceset="GND" device=""/>
+<part name="S2" library="switch-omron" deviceset="10-XX" device=""/>
+<part name="GND8" library="supply1" deviceset="GND" device=""/>
+<part name="X1" library="con-ptr500" deviceset="AK500/2" device=""/>
+<part name="X3" library="con-ptr500" deviceset="AK500/3" device=""/>
+<part name="GND9" library="supply1" deviceset="GND" device=""/>
+<part name="GND10" library="supply1" deviceset="GND" device=""/>
+<part name="P+6" library="supply1" deviceset="VCC" device=""/>
+<part name="X2" library="con-ptr500" deviceset="AK500/3" device=""/>
+<part name="P+7" library="supply1" deviceset="VCC" device=""/>
 </parts>
 <sheets>
@@
 <instance part="P+4" gate="VCC" x="25.4" y="91.44"/>
 <instance part="Q1" gate="G$1" x="17.78" y="55.88" rot="R90"/>
-<instance part="GND5" gate="1" x="17.78" y="43.18"/>
+<instance part="GND5" gate="1" x="25.4" y="45.72" rot="R270"/>
 <instance part="P+1" gate="VCC" x="25.4" y="35.56" rot="R180"/>
 <instance part="GND6" gate="1" x="-2.54" y="53.34"/>
@@
 <instance part="P+5" gate="VCC" x="121.92" y="10.16"/>
 <instance part="GND4" gate="1" x="121.92" y="-2.54"/>
+<instance part="S2" gate="1" x="63.5" y="99.06" rot="R270"/>
+<instance part="GND8" gate="1" x="73.66" y="91.44"/>
+<instance part="X1" gate="-1" x="96.52" y="106.68" rot="R270"/>
+<instance part="X1" gate="-2" x="91.44" y="106.68" rot="R270"/>
+<instance part="X3" gate="-1" x="180.34" y="43.18" rot="R180"/>
+<instance part="X3" gate="-2" x="180.34" y="48.26" rot="R180"/>
+<instance part="X3" gate="-3" x="180.34" y="53.34" rot="R180"/>
+<instance part="GND9" gate="1" x="170.18" y="35.56"/>
+<instance part="GND10" gate="1" x="96.52" y="93.98"/>
+<instance part="P+6" gate="VCC" x="91.44" y="93.98" rot="R180"/>
+<instance part="X2" gate="-1" x="180.34" y="10.16" rot="R180"/>
+<instance part="X2" gate="-2" x="180.34" y="15.24" rot="R180"/>
+<instance part="X2" gate="-3" x="180.34" y="20.32" rot="R180"/>
+<instance part="P+7" gate="VCC" x="170.18" y="25.4"/>
 </instances>
 <busses>
@@
 <pinref part="GND5" gate="1" pin="GND"/>
 <pinref part="IC2" gate="G$1" pin="GND@1"/>
-<wire x1="17.78" y1="45.72" x2="30.48" y2="45.72" width="0.1524" layer="91"/>
+<wire x1="27.94" y1="45.72" x2="30.48" y2="45.72" width="0.1524" layer="91"/>
 </segment>
 <segment>
@@
 <wire x1="109.22" y1="0" x2="121.92" y2="0" width="0.1524" layer="91"/>
 </segment>
+<segment>
+<pinref part="S2" gate="1" pin="S"/>
+<pinref part="S2" gate="1" pin="S1"/>
+<wire x1="68.58" y1="99.06" x2="68.58" y2="96.52" width="0.1524" layer="91"/>
+<pinref part="GND8" gate="1" pin="GND"/>
+<wire x1="68.58" y1="96.52" x2="73.66" y2="96.52" width="0.1524" layer="91"/>
+<wire x1="73.66" y1="96.52" x2="73.66" y2="93.98" width="0.1524" layer="91"/>
+<junction x="68.58" y="96.52"/>
+</segment>
+<segment>
+<pinref part="X3" gate="-1" pin="KL"/>
+<pinref part="GND9" gate="1" pin="GND"/>
+<wire x1="175.26" y1="43.18" x2="170.18" y2="43.18" width="0.1524" layer="91"/>
+<wire x1="170.18" y1="43.18" x2="170.18" y2="40.64" width="0.1524" layer="91"/>
+<pinref part="X2" gate="-1" pin="KL"/>
+<wire x1="170.18" y1="40.64" x2="170.18" y2="38.1" width="0.1524" layer="91"/>
+<wire x1="175.26" y1="10.16" x2="175.26" y2="5.08" width="0.1524" layer="91"/>
+<wire x1="175.26" y1="5.08" x2="195.58" y2="5.08" width="0.1524" layer="91"/>
+<wire x1="195.58" y1="5.08" x2="195.58" y2="38.1" width="0.1524" layer="91"/>
+<wire x1="195.58" y1="38.1" x2="172.72" y2="38.1" width="0.1524" layer="91"/>
+<wire x1="172.72" y1="38.1" x2="172.72" y2="40.64" width="0.1524" layer="91"/>
+<wire x1="172.72" y1="40.64" x2="170.18" y2="40.64" width="0.1524" layer="91"/>
+<junction x="170.18" y="40.64"/>
+</segment>
+<segment>
+<pinref part="X1" gate="-1" pin="KL"/>
+<pinref part="GND10" gate="1" pin="GND"/>
+<wire x1="96.52" y1="101.6" x2="96.52" y2="96.52" width="0.1524" layer="91"/>
+</segment>
 </net>
 <net name="N$5" class="0">
@@
 <wire x1="109.22" y1="5.08" x2="121.92" y2="5.08" width="0.1524" layer="91"/>
 <wire x1="121.92" y1="5.08" x2="121.92" y2="7.62" width="0.1524" layer="91"/>
+</segment>
+<segment>
+<pinref part="X1" gate="-2" pin="KL"/>
+<pinref part="P+6" gate="VCC" pin="VCC"/>
+<wire x1="91.44" y1="101.6" x2="91.44" y2="96.52" width="0.1524" layer="91"/>
+</segment>
+<segment>
+<pinref part="P+7" gate="VCC" pin="VCC"/>
+<wire x1="170.18" y1="22.86" x2="170.18" y2="20.32" width="0.1524" layer="91"/>
+<pinref part="X2" gate="-3" pin="KL"/>
+<wire x1="170.18" y1="20.32" x2="175.26" y2="20.32" width="0.1524" layer="91"/>
 </segment>
 </net>
@@
 <wire x1="30.48" y1="86.36" x2="30.48" y2="76.2" width="0.1524" layer="91"/>
 <junction x="30.48" y="76.2"/>
+<wire x1="53.34" y1="86.36" x2="55.88" y2="86.36" width="0.1524" layer="91"/>
+<wire x1="55.88" y1="86.36" x2="55.88" y2="96.52" width="0.1524" layer="91"/>
+<junction x="53.34" y="86.36"/>
+<pinref part="S2" gate="1" pin="P"/>
+<wire x1="55.88" y1="96.52" x2="55.88" y2="99.06" width="0.1524" layer="91"/>
+<wire x1="55.88" y1="99.06" x2="58.42" y2="99.06" width="0.1524" layer="91"/>
+<pinref part="S2" gate="1" pin="P1"/>
+<wire x1="58.42" y1="96.52" x2="55.88" y2="96.52" width="0.1524" layer="91"/>
+<junction x="55.88" y="96.52"/>
 </segment>
 </net>
@@
 </segment>
 </net>
+<net name="N$15" class="0">
+<segment>
+<pinref part="X3" gate="-3" pin="KL"/>
+<pinref part="IC1" gate="G$1" pin="B"/>
+<wire x1="175.26" y1="53.34" x2="167.64" y2="53.34" width="0.1524" layer="91"/>
+</segment>
+</net>
+<net name="N$16" class="0">
+<segment>
+<pinref part="IC1" gate="G$1" pin="A"/>
+<pinref part="X3" gate="-2" pin="KL"/>
+<wire x1="167.64" y1="48.26" x2="175.26" y2="48.26" width="0.1524" layer="91"/>
+</segment>
+</net>
+<net name="N$10" class="0">
+<segment>
+<pinref part="X2" gate="-2" pin="KL"/>
+<wire x1="175.26" y1="15.24" x2="101.6" y2="15.24" width="0.1524" layer="91"/>
+<wire x1="101.6" y1="15.24" x2="101.6" y2="25.4" width="0.1524" layer="91"/>
+<wire x1="101.6" y1="25.4" x2="83.82" y2="25.4" width="0.1524" layer="91"/>
+<wire x1="83.82" y1="25.4" x2="83.82" y2="45.72" width="0.1524" layer="91"/>
+<pinref part="IC2" gate="G$1" pin="PD3(INT1)"/>
+<wire x1="83.82" y1="45.72" x2="78.74" y2="45.72" width="0.1524" layer="91"/>
+</segment>
+</net>

Commit message: terrena
pcb
Parts:
- removed OK1, OK2: 4N25M, optocoupler:4N25M
- removed R3, R4, R5: (no value), rcl:R-EU_0204/7
- removed S2: (no value), switch-omron:10-XX
- added D1, D2: SFH482, led:SFH482
- added D3: 1N4004, diode:1N4004
- added R3_TX: (no value), rcl:R-EU_0204/7
- C1, C2: value (none) -> 22nf
- C3: value (none) -> .1nf
- Q1: value (none) -> 16mhz
- renumbered R2 to R2_RX, X1 to VCC, X2 to SENSOR, X3 to RS485
Connections:
- removed net N$16: IC1G$1.A, RS485-2.KL
- net GND: no longer OK1.C, OK2.C, R2_RX.2, R5.2, S2.S, S2.S1
- net N$10: now also IC2.PB0(ICP); no longer IC2.PD3(INT1)
- net N$13: no longer S2.P, S2.P1
- net N$15: now also D3.A, VCC-2.KL; no longer IC1G$1.B, RS485-3.KL
- net N$3: now also D1.C, IC2.PD0(RXD); no longer R4.1
- net N$4: now also D1.A, R2_RX.1; no longer OK1.A, R4.2
- net N$5: now also D2.A, R3_TX.1; no longer IC2.PD0(RXD), OK1.EMI, R2_RX.1
- net N$6: now also D2.C, IC1G$1.DI; no longer R3.2
- net N$7: now also IC1G$1.B, RS485-2.KL; no longer OK2.A, R3.1
- net N$8: now also IC1G$1.A, RS485-3.KL; no longer IC1G$1.DI, OK2.EMI, R5.1
- net VCC: now also D3.C, IC2.AVCC, R2_RX.2, R3_TX.2; no longer OK1.COL, OK2.COL, VCC-2.KL

Commit message: fix terrena
Parts:
- removed D2: SFH482, led:SFH482
- removed D3: 1N4004, diode:1N4004
- added LED_R2, LED_R3, LED_VCC: SFH482, led:SFH482
- added R_LED: (no value), rcl:R-EU_0204/7
- D1: value SFH482 -> 1N4004; device led:SFH482 -> diode:1N4004
Connections:
- new net N$17: LED_VCC.C, R_LED.1
- net GND: now also R_LED.2, SENSOR-3.KL; no longer RS485-1.KL, SENSOR-1.KL
- net N$10: now also SENSOR-1.KL; no longer SENSOR-2.KL
- net N$15: now also D1.A, LED_VCC.A; no longer D3.A
- net N$3: now also R2_RX.1; no longer D1.C
- net N$4: now also LED_R2.C, R2_RX.2; no longer D1.A, R2_RX.1
- net N$5: now also LED_R3.C, R3_TX.2; no longer D2.A, R3_TX.1
- net N$6: now also R3_TX.1; no longer D2.C
- net VCC: now also D1.C, LED_R2.A, LED_R3.A, SENSOR-2.KL; no longer D3.C, R2_RX.2, R3_TX.2, SENSOR-3.KL
Other:
- moved on the sheet: R2_RX, R3_TX

Commit message: fix
Parts:
- added JP2: (no value), pinhead:PINHD-2X3
Connections:
- net GND: now also JP2.6
Changed lines of the file:
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@@
 <grid distance="0.1" unitdist="inch" unit="inch" style="lines" multiple="1" display="no" altdistance="0.01" altunitdist="inch" altunit="inch"/>
 <layers>
-<layer number="1" name="Top" color="4" fill="1" visible="yes" active="no"/>
-<layer number="2" name="Route2" color="1" fill="3" visible="yes" active="no"/>
-<layer number="3" name="Route3" color="4" fill="3" visible="yes" active="no"/>
-<layer number="4" name="Route4" color="1" fill="4" visible="yes" active="no"/>
-<layer number="5" name="Route5" color="4" fill="4" visible="yes" active="no"/>
-<layer number="6" name="Route6" color="1" fill="8" visible="yes" active="no"/>
-<layer number="7" name="Route7" color="4" fill="8" visible="yes" active="no"/>
-<layer number="8" name="Route8" color="1" fill="2" visible="yes" active="no"/>
-<layer number="9" name="Route9" color="4" fill="2" visible="yes" active="no"/>
-<layer number="10" name="Route10" color="1" fill="7" visible="yes" active="no"/>
-<layer number="11" name="Route11" color="4" fill="7" visible="yes" active="no"/>
-<layer number="12" name="Route12" color="1" fill="5" visible="yes" active="no"/>
-<layer number="13" name="Route13" color="4" fill="5" visible="yes" active="no"/>
-<layer number="14" name="Route14" color="1" fill="6" visible="yes" active="no"/>
-<layer number="15" name="Route15" color="4" fill="6" visible="yes" active="no"/>
-<layer number="16" name="Bottom" color="1" fill="1" visible="yes" active="no"/>
-<layer number="17" name="Pads" color="2" fill="1" visible="yes" active="no"/>
-<layer number="18" name="Vias" color="2" fill="1" visible="yes" active="no"/>
-<layer number="19" name="Unrouted" color="6" fill="1" visible="yes" active="no"/>
-<layer number="20" name="Dimension" color="15" fill="1" visible="yes" active="no"/>
-<layer number="21" name="tPlace" color="7" fill="1" visible="yes" active="no"/>
-<layer number="22" name="bPlace" color="7" fill="1" visible="yes" active="no"/>
-<layer number="23" name="tOrigins" color="15" fill="1" visible="yes" active="no"/>
-<layer number="24" name="bOrigins" color="15" fill="1" visible="yes" active="no"/>
-<layer number="25" name="tNames" color="7" fill="1" visible="yes" active="no"/>
-<layer number="26" name="bNames" color="7" fill="1" visible="yes" active="no"/>
-<layer number="27" name="tValues" color="7" fill="1" visible="yes" active="no"/>
-<layer number="28" name="bValues" color="7" fill="1" visible="yes" active="no"/>
+<layer number="1" name="Top" color="4" fill="1" visible="no" active="no"/>
+<layer number="2" name="Route2" color="1" fill="3" visible="no" active="no"/>
+<layer number="3" name="Route3" color="4" fill="3" visible="no" active="no"/>
+<layer number="4" name="Route4" color="1" fill="4" visible="no" active="no"/>
+<layer number="5" name="Route5" color="4" fill="4" visible="no" active="no"/>
+<layer number="6" name="Route6" color="1" fill="8" visible="no" active="no"/>
+<layer number="7" name="Route7" color="4" fill="8" visible="no" active="no"/>
+<layer number="8" name="Route8" color="1" fill="2" visible="no" active="no"/>
+<layer number="9" name="Route9" color="4" fill="2" visible="no" active="no"/>
+<layer number="10" name="Route10" color="1" fill="7" visible="no" active="no"/>
+<layer number="11" name="Route11" color="4" fill="7" visible="no" active="no"/>
+<layer number="12" name="Route12" color="1" fill="5" visible="no" active="no"/>
+<layer number="13" name="Route13" color="4" fill="5" visible="no" active="no"/>
+<layer number="14" name="Route14" color="1" fill="6" visible="no" active="no"/>
+<layer number="15" name="Route15" color="4" fill="6" visible="no" active="no"/>
+<layer number="16" name="Bottom" color="1" fill="1" visible="no" active="no"/>
+<layer number="17" name="Pads" color="2" fill="1" visible="no" active="no"/>
+<layer number="18" name="Vias" color="2" fill="1" visible="no" active="no"/>
+<layer number="19" name="Unrouted" color="6" fill="1" visible="no" active="no"/>
+<layer number="20" name="Dimension" color="15" fill="1" visible="no" active="no"/>
+<layer number="21" name="tPlace" color="7" fill="1" visible="no" active="no"/>
+<layer number="22" name="bPlace" color="7" fill="1" visible="no" active="no"/>
+<layer number="23" name="tOrigins" color="15" fill="1" visible="no" active="no"/>
+<layer number="24" name="bOrigins" color="15" fill="1" visible="no" active="no"/>
+<layer number="25" name="tNames" color="7" fill="1" visible="no" active="no"/>
+<layer number="26" name="bNames" color="7" fill="1" visible="no" active="no"/>
+<layer number="27" name="tValues" color="7" fill="1" visible="no" active="no"/>
+<layer number="28" name="bValues" color="7" fill="1" visible="no" active="no"/>
 <layer number="29" name="tStop" color="7" fill="3" visible="no" active="no"/>
 <layer number="30" name="bStop" color="7" fill="6" visible="no" active="no"/>
@@
 <layer number="35" name="tGlue" color="7" fill="4" visible="no" active="no"/>
 <layer number="36" name="bGlue" color="7" fill="5" visible="no" active="no"/>
-<layer number="37" name="tTest" color="7" fill="1" visible="yes" active="no"/>
-<layer number="38" name="bTest" color="7" fill="1" visible="yes" active="no"/>
+<layer number="37" name="tTest" color="7" fill="1" visible="no" active="no"/>
+<layer number="38" name="bTest" color="7" fill="1" visible="no" active="no"/>
 <layer number="39" name="tKeepout" color="4" fill="11" visible="no" active="no"/>
 <layer number="40" name="bKeepout" color="1" fill="11" visible="no" active="no"/>
@@
 <layer number="44" name="Drills" color="7" fill="1" visible="no" active="no"/>
 <layer number="45" name="Holes" color="7" fill="1" visible="no" active="no"/>
-<layer number="46" name="Milling" color="3" fill="1" visible="yes" active="no"/>
-<layer number="47" name="Measures" color="7" fill="1" visible="yes" active="no"/>
-<layer number="48" name="Document" color="7" fill="1" visible="yes" active="no"/>
-<layer number="49" name="Reference" color="7" fill="1" visible="yes" active="no"/>
-<layer number="51" name="tDocu" color="7" fill="1" visible="yes" active="no"/>
-<layer number="52" name="bDocu" color="7" fill="1" visible="yes" active="no"/>
+<layer number="46" name="Milling" color="3" fill="1" visible="no" active="no"/>
+<layer number="47" name="Measures" color="7" fill="1" visible="no" active="no"/>
+<layer number="48" name="Document" color="7" fill="1" visible="no" active="no"/>
+<layer number="49" name="Reference" color="7" fill="1" visible="no" active="no"/>
+<layer number="51" name="tDocu" color="7" fill="1" visible="no" active="no"/>
+<layer number="52" name="bDocu" color="7" fill="1" visible="no" active="no"/>
 <layer number="90" name="Modules" color="5" fill="1" visible="yes" active="yes"/>
 <layer number="91" name="Nets" color="2" fill="1" visible="yes" active="yes"/>
@@
 <part name="R3_TX" library="rcl" deviceset="R-EU_" device="0204/7"/>
 <part name="D1" library="diode" deviceset="1N4004" device=""/>
+<part name="JP2" library="pinhead" deviceset="PINHD-2X3" device=""/>
 </parts>
 <sheets>
@@
 <instance part="R3_TX" gate="G$1" x="116.84" y="60.96" rot="R90"/>
 <instance part="D1" gate="1" x="81.28" y="99.06" rot="R180"/>
+<instance part="JP2" gate="A" x="142.24" y="0"/>
 </instances>
 <busses>
@@
 <pinref part="JP1" gate="A" pin="6"/>
 <pinref part="GND4" gate="1" pin="GND"/>
-<wire x1="109.22" y1="0" x2="121.92" y2="0" width="0.1524" layer="91"/>
-</segment>
-<segment>
+<wire x1="109.22" y1="0" x2="116.84" y2="0" width="0.1524" layer="91"/>
+<pinref part="JP2" gate="A" pin="6"/>
+<wire x1="116.84" y1="0" x2="121.92" y2="0" width="0.1524" layer="91"/>
+<wire x1="147.32" y1="-2.54" x2="157.48" y2="-2.54" width="0.1524" layer="91"/>
+<wire x1="157.48" y1="-2.54" x2="157.48" y2="-10.16" width="0.1524" layer="91"/>
+<wire x1="157.48" y1="-10.16" x2="116.84" y2="-10.16" width="0.1524" layer="91"/>
+<wire x1="116.84" y1="-10.16" x2="116.84" y2="0" width="0.1524" layer="91"/>
+</segment>
+<segment>

Commit message: FIX
Parts:
- renumbered JP1 to ISCP
Changed lines of the file:
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@@
 <part name="GND6" library="supply1" deviceset="GND" device=""/>
 <part name="GND7" library="supply1" deviceset="GND" device=""/>
-<part name="JP1" library="pinhead" deviceset="PINHD-2X3" device=""/>
+<part name="ISCP" library="pinhead" deviceset="PINHD-2X3" device=""/>
 <part name="P+5" library="supply1" deviceset="VCC" device=""/>
 <part name="GND4" library="supply1" deviceset="GND" device=""/>
@@
 <instance part="GND6" gate="1" x="-2.54" y="53.34"/>
 <instance part="GND7" gate="1" x="12.7" y="73.66"/>
-<instance part="JP1" gate="A" x="104.14" y="2.54"/>
+<instance part="ISCP" gate="A" x="104.14" y="2.54"/>
 <instance part="P+5" gate="VCC" x="121.92" y="10.16"/>
 <instance part="GND4" gate="1" x="121.92" y="-2.54"/>
@@
 </segment>
 <segment>
-<pinref part="JP1" gate="A" pin="6"/>
+<pinref part="ISCP" gate="A" pin="6"/>
 <pinref part="GND4" gate="1" pin="GND"/>
 <wire x1="109.22" y1="0" x2="116.84" y2="0" width="0.1524" layer="91"/>
@@
 </segment>
 <segment>
-<pinref part="JP1" gate="A" pin="2"/>
+<pinref part="ISCP" gate="A" pin="2"/>
 <pinref part="P+5" gate="VCC" pin="VCC"/>
 <wire x1="109.22" y1="5.08" x2="121.92" y2="5.08" width="0.1524" layer="91"/>
@@
 <pinref part="R1" gate="G$1" pin="1"/>
 <wire x1="30.48" y1="76.2" x2="25.4" y2="76.2" width="0.1524" layer="91"/>
-<pinref part="JP1" gate="A" pin="5"/>
+<pinref part="ISCP" gate="A" pin="5"/>
 <wire x1="101.6" y1="0" x2="53.34" y2="0" width="0.1524" layer="91"/>
 <wire x1="53.34" y1="0" x2="53.34" y2="86.36" width="0.1524" layer="91"/>
@@
 <wire x1="78.74" y1="20.32" x2="96.52" y2="20.32" width="0.1524" layer="91"/>
 <wire x1="96.52" y1="20.32" x2="96.52" y2="5.08" width="0.1524" layer="91"/>
-<pinref part="JP1" gate="A" pin="1"/>
+<pinref part="ISCP" gate="A" pin="1"/>
 <wire x1="96.52" y1="5.08" x2="101.6" y2="5.08" width="0.1524" layer="91"/>
 </segment>
@@
 <wire x1="78.74" y1="17.78" x2="93.98" y2="17.78" width="0.1524" layer="91"/>
 <wire x1="93.98" y1="17.78" x2="93.98" y2="2.54" width="0.1524" layer="91"/>
-<pinref part="JP1" gate="A" pin="3"/>
+<pinref part="ISCP" gate="A" pin="3"/>
 <wire x1="93.98" y1="2.54" x2="101.6" y2="2.54" width="0.1524" layer="91"/>
 </segment>
@@
 <net name="N$14" class="0">
 <segment>
-<pinref part="JP1" gate="A" pin="4"/>
+<pinref part="ISCP" gate="A" pin="4"/>
 <wire x1="109.22" y1="2.54" x2="116.84" y2="2.54" width="0.1524" layer="91"/>
 <wire x1="116.84" y1="2.54" x2="116.84" y2="22.86" width="0.1524" layer="91"/>
